File: hardware/v1.3/icepi-zero.kicad_sch (KiCad schematic)
At the start: 29 parts, among them J1 Conn_02x20_Counter_Clockwise, SW1 SW_Push, SW2 SW_Push, U1 ECP5-CABGA256, Y1 SG-8018CG 50.000000MHz

Commit message: QOL improvements on v1.3 PCB
Parts:
- LOGO1: value ~ -> (none)
